Commit message: Added detailed and simplified versions of URDF

File: Scripts/hexapod/urdf/hexapod_detailed.urdf (robot description, URDF)
Before this commit: robot hexapod, 19 links, 18 joints
Links:
- link base_link: geometry collision mesh filename=package://urdf/meshes/detailed/base_mesh.STL; visual mesh filename=package://urdf/meshes/detailed/base_mesh.STL
- link link_1_1: geometry collision mesh filename=package://urdf/meshes/detailed/coxa_mesh.STL; visual mesh filename=package://urdf/meshes/detailed/coxa_mesh.STL
- link link_1_2: geometry collision mesh filename=package://urdf/meshes/detailed/femur_mesh.STL; visual mesh filename=package://urdf/meshes/detailed/femur_mesh.STL
- link link_1_3: geometry collision mesh filename=package://urdf/meshes/detailed/tibia_mesh.STL; visual mesh filename=package://urdf/meshes/detailed/tibia_mesh.STL
- link link_2_1: geometry collision mesh filename=package://urdf/meshes/detailed/coxa_mesh.STL; visual mesh filename=package://urdf/meshes/detailed/coxa_mesh.STL
- link link_2_2: geometry collision mesh filename=package://urdf/meshes/detailed/femur_mesh.STL; visual mesh filename=package://urdf/meshes/detailed/femur_mesh.STL
- link link_2_3: geometry collision mesh filename=package://urdf/meshes/detailed/tibia_mesh.STL; visual mesh filename=package://urdf/meshes/detailed/tibia_mesh.STL
- link link_3_1: geometry collision mesh filename=package://urdf/meshes/detailed/coxa_mesh.STL; visual mesh filename=package://urdf/meshes/detailed/coxa_mesh.STL
- link link_3_2: geometry collision mesh filename=package://urdf/meshes/detailed/femur_mesh.STL; visual mesh filename=package://urdf/meshes/detailed/femur_mesh.STL
- link link_3_3: geometry collision mesh filename=package://urdf/meshes/detailed/tibia_mesh.STL; visual mesh filename=package://urdf/meshes/detailed/tibia_mesh.STL
- link link_4_1: geometry collision mesh filename=package://urdf/meshes/detailed/coxa_mesh.STL; visual mesh filename=package://urdf/meshes/detailed/coxa_mesh.STL
- link link_4_2: geometry collision mesh filename=package://urdf/meshes/detailed/femur_mesh.STL; visual mesh filename=package://urdf/meshes/detailed/femur_mesh.STL
- link link_4_3: geometry collision mesh filename=package://urdf/meshes/detailed/tibia_mesh.STL; visual mesh filename=package://urdf/meshes/detailed/tibia_mesh.STL
- link link_5_1: geometry collision mesh filename=package://urdf/meshes/detailed/coxa_mesh.STL; visual mesh filename=package://urdf/meshes/detailed/coxa_mesh.STL
- link link_5_2: geometry collision mesh filename=package://urdf/meshes/detailed/femur_mesh.STL; visual mesh filename=package://urdf/meshes/detailed/femur_mesh.STL
- link link_5_3: geometry collision mesh filename=package://urdf/meshes/detailed/tibia_mesh.STL; visual mesh filename=package://urdf/meshes/detailed/tibia_mesh.STL
- link link_6_1: geometry collision mesh filename=package://urdf/meshes/detailed/coxa_mesh.STL; visual mesh filename=package://urdf/meshes/detailed/coxa_mesh.STL
- link link_6_2: geometry collision mesh filename=package://urdf/meshes/detailed/femur_mesh.STL; visual mesh filename=package://urdf/meshes/detailed/femur_mesh.STL
- link link_6_3: geometry collision mesh filename=package://urdf/meshes/detailed/tibia_mesh.STL; visual mesh filename=package://urdf/meshes/detailed/tibia_mesh.STL
